File: hardware/kicad/xiao_esp32s3_breakout_board/xiao_esp32s3_breakout_board.kicad_pcb (KiCad board)
At the start: 2 copper layers, 50.8 x 38.1 mm, 11 parts, among them J1 XIAO_BREAKOUT_BOARD, J2 Conn_02x03_Odd_Even, J3 Conn_01x02_Pin, J4 Conn_01x07_Socket, J5 Conn_01x07_Socket

Commit message: これで注文した
Connections:
- J2 pad 1: unconnected-(J2-Pin_1-Pad1) -> /GPIO41_D12_MIC_DATA
- J2 pad 2: unconnected-(J2-Pin_2-Pad2) -> /GPIO40_CAM_SDA
- J2 pad 3: unconnected-(J2-Pin_3-Pad3) -> /CHIP_EN
- J2 pad 4: unconnected-(J2-Pin_4-Pad4) -> GND
- J2 pad 5: unconnected-(J2-Pin_5-Pad5) -> /GPIO42_D11_MIC_CLK
- J2 pad 6: unconnected-(J2-Pin_6-Pad6) -> /GPIO39_CAM_SCL
- J3 pad 1: unconnected-(J3-Pin_1-Pad1) -> GND
- J3 pad 2: unconnected-(J3-Pin_2-Pad2) -> +BATT
- J4 pad 1: unconnected-(J4-Pin_1-Pad1) -> /GPIO1_D0_A0
- J4 pad 2: unconnected-(J4-Pin_2-Pad2) -> /GPIO2_D1_A1
- J4 pad 3: unconnected-(J4-Pin_3-Pad3) -> /GPIO3_D2_A2
- J4 pad 4: unconnected-(J4-Pin_4-Pad4) -> /GPIO4_D3_A3
- J4 pad 5: unconnected-(J4-Pin_5-Pad5) -> /GPIO5_D4_A4_SDA
- J4 pad 6: unconnected-(J4-Pin_6-Pad6) -> /GPIO6_D5_A5_SCL
- J4 pad 7: unconnected-(J4-Pin_7-Pad7) -> /GPIO43_D6_TX
- J5 pad 1: unconnected-(J5-Pin_1-Pad1) -> VBUS
- J5 pad 2: unconnected-(J5-Pin_2-Pad2) -> GND
- J5 pad 3: unconnected-(J5-Pin_3-Pad3) -> 3V3
- J5 pad 4: unconnected-(J5-Pin_4-Pad4) -> /GPIO9_D10_A10_MOSI
- J5 pad 5: unconnected-(J5-Pin_5-Pad5) -> /GPIO8_D9_A9_MISO
- J5 pad 6: unconnected-(J5-Pin_6-Pad6) -> /GPIO7_D8_A8_SCK
- J5 pad 7: unconnected-(J5-Pin_7-Pad7) -> /GPIO44_D7_RX
Routing:
- net /GPIO39_CAM_SCL: track 0.00 -> 85.4 mm
- net /GPIO40_CAM_SDA: track 0.00 -> 72.0 mm
- net VBUS: track 0.00 -> 70.4 mm
- net +BATT: track 0.00 -> 65.2 mm
- net 3V3: track 0.00 -> 58.4 mm
- net /GPIO9_D10_A10_MOSI: track 0.00 -> 52.0 mm
- net /GPIO8_D9_A9_MISO: track 0.00 -> 45.4 mm
- net /GPIO2_D1_A1: track 0.00 -> 44.5 mm
- net /GPIO42_D11_MIC_CLK: track 0.00 -> 43.0 mm
- net /GPIO41_D12_MIC_DATA: track 0.00 -> 42.5 mm
- net /GPIO7_D8_A8_SCK: track 0.00 -> 39.6 mm
- net /GPIO1_D0_A0: track 0.00 -> 38.7 mm
- net /GPIO3_D2_A2: track 0.00 -> 38.0 mm
- net /GPIO4_D3_A3: track 0.00 -> 33.8 mm
- net /GPIO44_D7_RX: track 0.00 -> 33.8 mm
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- added copper zone on B.Cu, net GND
- added copper zone on F.Cu, net GND
Other:
- board text added: "+B"
- board text added: "+BAT"
- board text added: "-B"
- board text added: "3V3"
- board text added: "D0"
- board text added: "D1"
- board text added: "D10"
- board text added: "D11"
- board text added: "D12"
- board text added: "D2"
- board text added: "D3"
- board text added: "D4"
- board text added: "D5"
- board text added: "D6"
- board text added: "D7"
- board text added: "D8"
- board text added: "D9"
- board text added: "EN"
- board text added: "GND"
- board text added: "IO39"
- board text added: "IO40"
- board text added: "IO41"
- board text added: "IO42"
- board text added: "VBUS"
- board text added: "XIAO_ESP32S3_BREAKOUT_BOARD Rev1"
