File: hardware/kicad/xiao_esp32s3_breakout_board/xiao_esp32s3_breakout_board.kicad_sch (KiCad schematic)
At the start: 4 parts, among them J1 XIAO_BREAKOUT_BOARD, U1 XIAO-ESP32-S3

Commit message: ブレイクアウトボード作成中
Parts:
- added J2: Conn_02x03_Odd_Even, Connector_PinHeader_2.54mm:PinHeader_2x03_P2.54mm_Vertical, symbol Connector_Generic:Conn_02x03_Odd_Even
- added J3: Conn_01x02_Pin, Connector_PinHeader_2.00mm:PinHeader_1x02_P2.00mm_Vertical, symbol Connector:Conn_01x02_Pin
- added J4, J5: Conn_01x07_Socket, Connector_PinSocket_2.54mm:PinSocket_1x07_P2.54mm_Vertical, symbol Connector:Conn_01x07_Socket
- J1: footprint (none) -> Connector_IDC:IDC-Header_2x10_P2.54mm_Vertical
- TP1, TP2: footprint (none) -> TestPoint:TestPoint_THTPad_D1.5mm_Drill0.7mm
- U1: footprint Seeed_Studio_XIAO_Series:XIAO-ESP32-S3-SMD -> @自分用:XIAO-ESP32-S3-SMD
Connections:
- net +BATT: now also U1.23 (BAT+); no longer U1.32 (BAT+)
- net CHIP_EN: now also U1.17 (CHIP_EN); no longer U1.26 (CHIP_EN)
- net GND: now also U1.18 (GND), U1.24 (BAT-); no longer U1.27 (GND), U1.33 (BAT-)
- net GPIO39_CAM_SCL: now also U1.20 (GPIO39_MTCK); no longer U1.29 (GPIO39_MTCK)
- net GPIO40_CAM_SDA: now also U1.16 (GPIO40_MTDO); no longer U1.25 (GPIO40_MTDO)
- net GPIO41_D12_MIC_DATA: now also U1.15 (GPIO41_MTDI); no longer U1.24 (GPIO41_MTDI)
- net GPIO42_D11_MIC_CLK: now also U1.19 (GPIO42_MTMS); no longer U1.28 (GPIO42_MTMS)

Commit message: これで注文した
Parts:
- removed U1: XIAO-ESP32-S3, @自分用:XIAO-ESP32-S3-SMD, symbol Seeed_Studio_XIAO_Series:XIAO-ESP32-S3-SMD
Connections:
- net +BATT: now also J3.2 (Pin_2)
- net 3V3: now also J5.3 (Pin_3)
- net CHIP_EN: now also J2.3 (Pin_3)
- net GND: now also J2.4 (Pin_4), J3.1 (Pin_1), J5.2 (Pin_2)
- net GPIO1_D0_A0: now also J4.1 (Pin_1)
- net GPIO2_D1_A1: now also J4.2 (Pin_2)
- net GPIO39_CAM_SCL: now also J2.6 (Pin_6)
- net GPIO3_D2_A2: now also J4.3 (Pin_3)
- net GPIO40_CAM_SDA: now also J2.2 (Pin_2)
- net GPIO41_D12_MIC_DATA: now also J2.1 (Pin_1)
- net GPIO42_D11_MIC_CLK: now also J2.5 (Pin_5)
- net GPIO43_D6_TX: now also J4.7 (Pin_7)
- net GPIO44_D7_RX: now also J5.7 (Pin_7)
- net GPIO4_D3_A3: now also J4.4 (Pin_4)
- net GPIO5_D4_A4_SDA: now also J4.5 (Pin_5)
- net GPIO6_D5_A5_SCL: now also J4.6 (Pin_6)
- net GPIO7_D8_A8_SCK: now also J5.6 (Pin_6)
- net GPIO8_D9_A9_MISO: now also J5.5 (Pin_5)
- net GPIO9_D10_A10_MOSI: now also J5.4 (Pin_4)
- net VBUS: now also J5.1 (Pin_1)
- no-connect marks 3 -> 0
Other:
- moved on the sheet: J2, J3, J4, J5
